File: func/func.sch (KiCad schematic (older format))
At the start: 0 parts

Commit message: Частичная схемо
Parts:
- added R1 (x2), R3, R4, R5: 100k, symbol Device:R
- added SW? (x5): SW_MEC_5G, symbol Switch:SW_MEC_5G
- added U?: EXP, symbol FUNG:EXP
- added U?: PEVM, symbol FUNG:PEVM
Connections:
- net labels added: Earth, PD0, PD1, PD2, PD3, PD4, PD5
- wire segments 0 -> 28
Other:
- note added: "ИСТОЧНИК"
- note added: "ПОЛУЧАТЕЛЬ"

Commit message: Функц
Parts:
- removed U?: PEVM, symbol FUNG:PEVM
- added AFF?: LTS-6980HR, Display_7Segment:7SegmentLED_LTS6760_LTS6780, symbol Display_Character:LTS-6980HR
- added U?: rs232, symbol FUNG:rs232
- added U?: PEVM, symbol FUNG:PEVM
- added U?: prog, symbol FUNG:prog
- added U?: XRAM, symbol FUNG:XRAM
- added U?: EXP_copy, symbol FUNG:EXP_copy
- gave numbers to parts that had none: 5
Connections:
- net labels added: PB0
- net labels removed: PD0, PD1
- wire segments 28 -> 19
Other:
- note added: "PB1"
- note added: "PD0"
- note added: "PD1"

Commit message: ЗАМЕЧАНИЕ
Parts:
- removed R1 (x2), R3, R4, R5: 100k, symbol Device:R
Connections:
- wire segments 19 -> 14
Changed lines of the file:
@@
 	1    0    0    -1
 $EndComp
-$Comp
-L Device:R R1
-U 1 1 6189D65D
-P 8300 8600
-F 0 "R1" V 8507 8600 50  0000 C CNN
-F 1 "100k" V 8416 8600 50  0000 C CNN
-F 2 "" V 8230 8600 50  0001 C CNN
-F 3 "~" H 8300 8600 50  0001 C CNN
-	1    8300 8600
-	0    -1   -1   0
-$EndComp
-$Comp
-L Device:R R3
-U 1 1 6189EDB1
-P 8300 9000
-F 0 "R3" V 8507 9000 50  0000 C CNN
-F 1 "100k" V 8416 9000 50  0000 C CNN
-F 2 "" V 8230 9000 50  0001 C CNN
-F 3 "~" H 8300 9000 50  0001 C CNN
-	1    8300 9000
-	0    -1   -1   0
-$EndComp
-$Comp
-L Device:R R4
-U 1 1 6189F8F0
-P 8300 9400
-F 0 "R4" V 8507 9400 50  0000 C CNN
-F 1 "100k" V 8416 9400 50  0000 C CNN
-F 2 "" V 8230 9400 50  0001 C CNN
-F 3 "~" H 8300 9400 50  0001 C CNN
-	1    8300 9400
-	0    -1   -1   0
-$EndComp
-$Comp
-L Device:R R5
-U 1 1 618A04E8
-P 8300 9800
-F 0 "R5" V 8507 9800 50  0000 C CNN
-F 1 "100k" V 8416 9800 50  0000 C CNN
-F 2 "" V 8230 9800 50  0001 C CNN
-F 3 "~" H 8300 9800 50  0001 C CNN
-	1    8300 9800
-	0    -1   -1   0
-$EndComp
-Wire Wire Line
-	8050 8250 8150 8250
-Wire Wire Line
-	8150 8600 8050 8600
-Wire Wire Line
-	8050 9000 8150 9000
-Wire Wire Line
-	8150 9400 8050 9400
-Wire Wire Line
-	8050 9800 8150 9800
 Wire Bus Line
 	6700 1250 6700 4850
@@
 	13550 8750 13550 8450
 Connection ~ 13550 8450
-$Comp
-L Device:R R1
-U 1 1 6189C0E3
-P 8300 8250
-F 0 "R1" V 8507 8250 50  0000 C CNN
-F 1 "100k" V 8416 8250 50  0000 C CNN
-F 2 "" V 8230 8250 50  0001 C CNN
-F 3 "~" H 8300 8250 50  0001 C CNN
-	1    8300 8250
-	0    -1   -1   0
-$EndComp
-Wire Wire Line
-	8450 8250 8700 8250
 Entry Wire Line
 	8700 8250 8800 8350
 Text Label 8500 8250 0    50   ~ 0
 PB0
-Wire Wire Line
-	8450 8600 8700 8600
 Entry Wire Line
 	8700 8600 8800 8700
 Text Label 8500 8600 0    50   ~ 0
 PD2
-Wire Wire Line
-	8450 9000 8700 9000
 Entry Wire Line
 	8700 9000 8800 9100
 Text Label 8500 9000 0    50   ~ 0
 PD3
-Wire Wire Line
-	8450 9400 8700 9400
 Entry Wire Line
 	8700 9400 8800 9500
 Text Label 8500 9400 0    50   ~ 0
 PD4
-Wire Wire Line
-	8450 9800 8700 9800
 Entry Wire Line
 	8700 9800 8800 9900
@@
 Wire Wire Line
 	11400 8550 11400 8400
+Wire Wire Line
+	8050 8250 8700 8250
+Wire Wire Line
+	8050 8600 8700 8600
+Wire Wire Line
+	8050 9000 8700 9000
+Wire Wire Line
+	8050 9400 8700 9400
+Wire Wire Line
+	8050 9800 8700 9800
 Wire Bus Line
 	9650 8650 12050 8650

Commit message: Added components
Parts:
- removed U?: PEVM, symbol FUNG:PEVM
Other:
- note added: "К ПЭВМ"
Changed lines of the file:
@@
 	8050 7100 8150 7200
 Wire Bus Line
-	11800 8450 12050 8450
-Wire Bus Line
 	12050 8450 12050 8650
-Connection ~ 12050 8450
-Wire Bus Line
-	12050 8450 12250 8450
 Entry Wire Line
 	9550 4950 9650 5050
@@
 Wire Bus Line
 	6700 4850 8050 4850
-Wire Bus Line
-	13300 8450 13550 8450
 Entry Bus Bus
 	13550 8750 13650 8850
 Wire Bus Line
 	13550 8750 13550 8450
-Connection ~ 13550 8450
 Entry Wire Line
 	8700 8250 8800 8350
@@
 Entry Wire Line
 	11250 8750 11350 8850
-Wire Bus Line
-	13550 8450 14350 8450
-Connection ~ 8800 8850
-$Comp
-L FUNG:PEVM U?
-U 1 1 618A29A2
-P 16000 8450
-F 0 "U?" H 16228 8321 50  0001 L CNN
-F 1 "PEVM" H 16228 8275 50  0001 L CNN
-F 2 "" H 16000 8450 50  0001 C CNN
-F 3 "" H 16000 8450 50  0001 C CNN
-	1    16000 8450
-	1    0    0    -1
-$EndComp
 $Comp
 L FUNG:rs232 U?
@@
 Wire Bus Line
 	8900 4050 8950 4050
-Wire Bus Line
-	8950 4050 8950 4150
-Connection ~ 8950 4050
 Text Notes 7050 4300 0    50   ~ 0
 PB1
@@
 Wire Wire Line
 	8050 9800 8700 9800
+Text Notes 15700 8700 0    50   ~ 0
+К ПЭВМ
+Wire Bus Line
+	8950 4050 8950 4150
+Wire Bus Line
+	13300 8450 14350 8450
+Wire Bus Line
+	11800 8450 12250 8450
+Entry Bus Bus
+	8800 8950 8900 8850
 Wire Bus Line
 	9650 8650 12050 8650
@@
 	1900 1800 3050 1800
 Wire Bus Line
-	8800 8150 8800 8850
-Wire Bus Line
 	8450 450  13350 450
 Wire Bus Line
 	1850 1250 6700 1250
-Wire Bus Line
-	8800 8850 8800 10000
-Wire Bus Line
-	8800 8850 14300 8850
 Wire Wire Line
 	7550 8150 7550 9950
@@
 	8950 3550 8950 4050
 Wire Bus Line
+	8900 8850 14300 8850
+Wire Bus Line
 	9650 4700 9650 8650
 Wire Bus Line
+	8800 8150 8800 10000
+Wire Bus Line
 	7150 7700 7150 10950

Commit message: New schematics alpha
Parts:
- removed AFF?: LTS-6980HR, Display_7Segment:7SegmentLED_LTS6760_LTS6780, symbol Display_Character:LTS-6980HR
- removed U?: EXP_copy, symbol FUNG:EXP_copy
- added C? (x2): C, symbol Device:C
- added U?: cmp_internal, symbol FUNG:cmp_internal
- added U?: CPU, symbol FUNG:CPU
- added U?: EEPROM, symbol FUNG:EEPROM
- added U?: INTERRUPTS, symbol FUNG:INTERRUPTS
- added U?: MCU_TIMERS, symbol FUNG:MCU_TIMERS
- added U?: OSC_INT, symbol FUNG:OSC_INT
- added U?: PORTA, symbol FUNG:PORTA
- added U?: PORTB, symbol FUNG:PORTB
- added U?: PORTC, symbol FUNG:PORTC
- added U?: PORTD, symbol FUNG:PORTD
- added U?: PORTE, symbol FUNG:PORTE
- added U?: prog_logic, symbol FUNG:prog_logic
- added U?: SPI, symbol FUNG:SPI
- added U?: USART, symbol FUNG:USART
- added U?: WATCHDOG, symbol FUNG:WATCHDOG
- added U?: XTAL, symbol FUNG:XTAL
- added U?: XTAL_int, symbol FUNG:XTAL_int
- added Y?: XTAL1, symbol Device:Crystal
Connections:
- net labels added: PA0, PA1, PA2
- wire segments 14 -> 38
Other:
- note added: "XTAL1"
- note added: "XTAL2"
- note added: "~RESET"
- note removed: "PB1"
- note removed: "PD0"
- note removed: "PD1"
- note removed: "ИСТОЧНИК"
- moved on the sheet: SW1, SW2, SW3, SW4, SW5

Commit message: More schematics
Parts:
- added U?: CA56-12CGKWA, Display_7Segment:CA56-12CGKWA, symbol Display_Character:CA56-12CGKWA
Connections:
- net labels added: PA3, PA4, PA5, PA6, PA7
- wire segments 38 -> 76
Other:
- moved on the sheet: U?

Commit message: Finished port labeling
Connections:
- net labels added: PB1, PB2, PB3, PB4, PB5, PB6, PB7, PC0, PC1, PC2, PC3, PC4, PC5, PC6, PC7, PD0, PD1, PD6, PD7
Changed lines of the file:
@@
 	14100 2500 14100 2250
 Text Label 13400 2450 1    50   ~ 0
-PA0
+PC0
 Text Label 13500 2450 1    50   ~ 0
-PA1
+PC1
 Text Label 13600 2450 1    50   ~ 0
-PA2
+PC2
 Text Label 13700 2450 1    50   ~ 0
-PA3
+PC3
 Text Label 13800 2450 1    50   ~ 0
-PA4
+PC4
 Text Label 13900 2450 1    50   ~ 0
-PA5
+PC5
 Text Label 14000 2450 1    50   ~ 0
-PA6
+PC6
 Text Label 14100 2450 1    50   ~ 0
-PA7
-Wire Wire Line
-	12050 7700 12050 7450
-Wire Wire Line
-	11950 7450 11950 7700
-Wire Wire Line
-	11850 7450 11850 7700
-Wire Wire Line
-	11750 7450 11750 7700
-Wire Wire Line
-	11650 7450 11650 7700
-Wire Wire Line
-	11550 7450 11550 7700
-Wire Wire Line
-	11450 7450 11450 7700
-Wire Wire Line
-	11350 7450 11350 7700
-Text Label 12050 7500 3    50   ~ 0
-PA0
-Text Label 11950 7500 3    50   ~ 0
-PA1
-Text Label 11850 7500 3    50   ~ 0
-PA2
-Text Label 11750 7500 3    50   ~ 0
-PA3
-Text Label 11650 7500 3    50   ~ 0
-PA4
-Text Label 11550 7500 3    50   ~ 0
-PA5
-Text Label 11450 7500 3    50   ~ 0
-PA6
-Text Label 11350 7500 3    50   ~ 0
-PA7
+PC7
 Wire Wire Line
 	13450 7450 13450 7700
@@
 	14150 7700 14150 7450
 Text Label 13450 7650 1    50   ~ 0
-PA0
+PD0
 Text Label 13550 7650 1    50   ~ 0
-PA1
+PD1
 Text Label 13650 7650 1    50   ~ 0
-PA2
+PD2
 Text Label 13750 7650 1    50   ~ 0
-PA3
+PD3
 Text Label 13850 7650 1    50   ~ 0
-PA4
+PD4
 Text Label 13950 7650 1    50   ~ 0
-PA5
+PD5
 Text Label 14050 7650 1    50   ~ 0
-PA6
+PD6
 Text Label 14150 7650 1    50   ~ 0
-PA7
+PD7
 Wire Wire Line
 	11900 7000 11900 7150
@@
 Wire Wire Line
 	13800 7000 13800 7150
-Wire Bus Line
-	11400 7000 14100 7000
-Wire Bus Line
-	11250 3050 14000 3050
-Wire Bus Line
-	13350 750  14350 750
-Wire Bus Line
-	8350 1350 8350 3250
-Wire Bus Line
-	8450 450  13350 450
-Wire Wire Line
-	4700 7750 4700 9550
-Wire Bus Line
-	6500 7750 6500 9600
-Wire Bus Line
-	3300 7550 3300 10800
-Wire Bus Line
-	8350 550  8350 1300
-Wire Bus Line
-	3400 4100 3400 6400
 $Comp
 L Graphic:SYM_Arrow_Tiny #SYM?
@@
 	0    -1   -1   0
 $EndComp
+Wire Wire Line
+	11350 7450 11350 7700
+Wire Wire Line
+	11450 7700 11450 7450
+Wire Wire Line
+	11550 7700 11550 7450
+Wire Wire Line
+	11650 7700 11650 7450
+Wire Wire Line
+	11750 7700 11750 7450
+Wire Wire Line
+	11850 7700 11850 7450
+Wire Wire Line
+	11950 7700 11950 7450
+Wire Wire Line
+	12050 7700 12050 7450
+Text Label 11350 7650 1    50   ~ 0
+PB0
+Text Label 11450 7650 1    50   ~ 0
+PB1
+Text Label 11550 7650 1    50   ~ 0
+PB2
+Text Label 11650 7650 1    50   ~ 0
+PB3
+Text Label 11750 7650 1    50   ~ 0
+PB4
+Text Label 11850 7650 1    50   ~ 0
+PB5
+Text Label 11950 7650 1    50   ~ 0
+PB6
+Text Label 12050 7650 1    50   ~ 0
+PB7
+Wire Bus Line
+	11400 7000 14100 7000
+Wire Bus Line
+	11250 3050 14000 3050
+Wire Bus Line
+	13350 750  14350 750
+Wire Bus Line
+	8350 1350 8350 3250
+Wire Bus Line
+	8450 450  13350 450
+Wire Wire Line
+	4700 7750 4700 9550
+Wire Bus Line
+	6500 7750 6500 9600
+Wire Bus Line
+	3300 7550 3300 10800
+Wire Bus Line
+	8350 550  8350 1300
+Wire Bus Line
+	3400 4100 3400 6400
 $EndSCHEMATC

Commit message: Finished port labeling
Parts:
- added U?: Driver_TM1637, symbol kur_func:Driver_TM1637
Connections:
- net labels added: DIO, GRID1, GRID2, GRID3, GRID4, GRID5, GRID6, K1, K2, VCC
- wire segments 76 -> 120
Other:
- note added: "CLK"
Changed lines of the file:
@@
 U 1 1 61A5A1CF
 P 12100 5250
-F 0 "U?" H 12378 5055 50  0000 L CNN
+F 0 "U?" H 12378 5055 50  0001 L CNN
 F 1 "cmp_internal" H 12100 5250 50  0001 C CNN
 F 2 "" H 12100 5250 50  0001 C CNN
@@
 U 1 1 61A5AC5D
 P 12100 3800
-F 0 "U?" H 12378 3600 50  0000 L CNN
+F 0 "U?" H 12378 3600 50  0001 L CNN
 F 1 "CPU" H 12100 3800 50  0001 C CNN
 F 2 "" H 12100 3800 50  0001 C CNN
@@
 U 1 1 61A5B4D9
 P 13300 5550
-F 0 "U?" H 13578 5350 50  0000 L CNN
+F 0 "U?" H 13578 5350 50  0001 L CNN
 F 1 "EEPROM" H 13300 5550 50  0001 C CNN
 F 2 "" H 13300 5550 50  0001 C CNN
@@
 U 1 1 61A5BC51
 P 13300 4950
-F 0 "U?" H 13578 4750 50  0000 L CNN
+F 0 "U?" H 13578 4750 50  0001 L CNN
 F 1 "INTERRUPTS" H 13300 4950 50  0001 C CNN
 F 2 "" H 13300 4950 50  0001 C CNN
@@
 U 1 1 61A5C2CE
 P 13300 4350
-F 0 "U?" H 13578 4150 50  0000 L CNN
+F 0 "U?" H 13578 4150 50  0001 L CNN
 F 1 "MCU_TIMERS" H 13300 4350 50  0001 C CNN
 F 2 "" H 13300 4350 50  0001 C CNN
@@
 U 1 1 61A5C968
 P 13300 3250
-F 0 "U?" H 13578 3050 50  0000 L CNN
+F 0 "U?" H 13578 3050 50  0001 L CNN
 F 1 "OSC_INT" H 13300 3250 50  0001 C CNN
 F 2 "" H 13300 3250 50  0001 C CNN
@@
 U 1 1 61A5D059
 P 11550 2450
-F 0 "U?" H 11928 2250 50  0000 L CNN
+F 0 "U?" H 11928 2250 50  0001 L CNN
 F 1 "PORTA" H 11550 2450 50  0001 C CNN
 F 2 "" H 11550 2450 50  0001 C CNN
@@
 U 1 1 61A5DA97
 P 11700 7100
-F 0 "U?" H 12078 6900 50  0000 L CNN
+F 0 "U?" H 12078 6900 50  0001 L CNN
 F 1 "PORTB" H 11700 7100 50  0001 C CNN
 F 2 "" H 11700 7100 50  0001 C CNN
@@
 U 1 1 61A5E2AF
 P 13750 2450
-F 0 "U?" H 14128 2250 50  0000 L CNN
+F 0 "U?" H 14128 2250 50  0001 L CNN
 F 1 "PORTC" H 13750 2450 50  0001 C CNN
 F 2 "" H 13750 2450 50  0001 C CNN
@@
 U 1 1 61A5EA11
 P 13800 7100
-F 0 "U?" H 14178 6900 50  0000 L CNN
+F 0 "U?" H 14178 6900 50  0001 L CNN
 F 1 "PORTD" H 13800 7100 50  0001 C CNN
 F 2 "" H 13800 7100 50  0001 C CNN
@@
 U 1 1 61A5F0EC
 P 12650 2450
-F 0 "U?" H 12878 2250 50  0000 L CNN
+F 0 "U?" H 12878 2250 50  0001 L CNN
 F 1 "PORTE" H 12650 2450 50  0001 C CNN
 F 2 "" H 12650 2450 50  0001 C CNN
@@
 U 1 1 61A60964
 P 13300 6200
-F 0 "U?" H 13578 6000 50  0000 L CNN
+F 0 "U?" H 13578 6000 50  0001 L CNN
 F 1 "USART" H 13300 6200 50  0001 C CNN
 F 2 "" H 13300 6200 50  0001 C CNN
@@
 U 1 1 61A61309
 P 13300 3800
-F 0 "U?" H 13578 3600 50  0000 L CNN
+F 0 "U?" H 13578 3600 50  0001 L CNN
 F 1 "WATCHDOG" H 13300 3800 50  0001 C CNN
 F 2 "" H 13300 3800 50  0001 C CNN
@@
 U 1 1 61A6209D
 P 14250 3800
-F 0 "U?" H 14528 3600 50  0000 L CNN
+F 0 "U?" H 14528 3600 50  0001 L CNN
 F 1 "XTAL" H 14250 3800 50  0001 C CNN
 F 2 "" H 14250 3800 50  0001 C CNN
@@
 U 1 1 61B45411
 P 14250 4750
-F 0 "U?" H 14578 4500 50  0000 L CNN
+F 0 "U?" H 14578 4500 50  0001 L CNN
 F 1 "XTAL_int" H 14250 4750 50  0001 C CNN
 F 2 "" H 14250 4750 50  0001 C CNN
@@
 L Display_Character:CA56-12CGKWA U?
 U 1 1 61A67960
-P 8450 5050
-F 0 "U?" H 8450 5717 50  0000 C CNN
-F 1 "CA56-12CGKWA" H 8450 5626 50  0000 C CNN
-F 2 "Display_7Segment:CA56-12CGKWA" H 8450 4450 50  0001 C CNN
-F 3 "http://www.kingbright.com/attachments/file/psearch/000/00/00/CA56-12CGKWA(Ver.9A).pdf" H 8020 5080 50  0001 C CNN
-	1    8450 5050
+P 8800 5050
+F 0 "U?" H 8800 5717 50  0001 C CNN
+F 1 "CA56-12CGKWA" H 8800 5626 50  0001 C CNN
+F 2 "Display_7Segment:CA56-12CGKWA" H 8800 4450 50  0001 C CNN
+F 3 "http://www.kingbright.com/attachments/file/psearch/000/00/00/CA56-12CGKWA(Ver.9A).pdf" H 8370 5080 50  0001 C CNN
+	1    8800 5050
 	1    0    0    -1
 $EndComp
@@
 	11450 7700 11450 7450
 Wire Wire Line
-	11550 7700 11550 7450
-Wire Wire Line
-	11650 7700 11650 7450
+	11550 7700 11550 7600
+Wire Wire Line
+	11650 7700 11650 7500
 Wire Wire Line
 	11750 7700 11750 7450
@@
 Text Label 12050 7650 1    50   ~ 0
 PB7
+Wire Wire Line
+	11750 5350 10500 5350
+Wire Wire Line
+	10500 5350 10500 7600
+Wire Wire Line
+	10500 7600 11550 7600
+Connection ~ 11550 7600
+Wire Wire Line
+	11550 7600 11550 7450
+Wire Wire Line
+	11750 5550 10600 5550
+Wire Wire Line
+	10600 5550 10600 7500
+Wire Wire Line
+	10600 7500 11650 7500
+Connection ~ 11650 7500
+Wire Wire Line
+	11650 7500 11650 7450
+$Comp
+L kur_func:Driver_TM1637 U?
+U 1 1 61A782A3
+P 6450 6350
+F 0 "U?" H 6483 7115 50  0000 C CNN
+F 1 "Driver_TM1637" H 6483 7024 50  0000 C CNN
+F 2 "" H 6100 7250 50  0001 C CNN
+F 3 "" H 6100 7250 50  0001 C CNN
+	1    6450 6350
+	1    0    0    -1
+$EndComp
+Wire Wire Line
+	7050 5850 7250 5850
+Wire Wire Line
+	7050 6750 7250 6750
+Wire Wire Line
+	7050 6850 7250 6850
+Wire Wire Line
+	7250 5850 7250 4750
+Wire Wire Line
+	7250 4750 7700 4750
+Wire Wire Line
+	7700 4850 7300 4850
+Wire Wire Line
+	7300 4850 7300 5950
+Wire Wire Line
+	7050 5950 7300 5950
+Wire Wire Line
+	7350 6050 7350 4950
+Wire Wire Line
+	7350 4950 7700 4950
+Wire Wire Line
+	7050 6050 7350 6050
+Wire Wire Line
+	7700 5050 7400 5050
+Wire Wire Line
+	7400 5050 7400 6150
+Wire Wire Line
+	7050 6150 7400 6150
+Wire Wire Line
+	7700 5150 7450 5150
+Wire Wire Line
+	7450 5150 7450 6250
+Wire Wire Line
+	7050 6250 7450 6250
+Wire Wire Line
+	7500 6350 7500 5250
+Wire Wire Line
+	7500 5250 7700 5250
+Wire Wire Line
+	7050 6350 7500 6350
+Wire Wire Line
+	7700 5350 7550 5350
+Wire Wire Line
+	7550 5350 7550 6450
+Wire Wire Line
+	7050 6450 7550 6450
+Wire Wire Line
+	7600 6550 7600 5450
+Wire Wire Line
+	7600 5450 7700 5450
+Wire Wire Line
+	7050 6550 7600 6550
+$Comp
+L power:VCC #PWR?
+U 1 1 61AD6DB8
+P 7250 6750
+F 0 "#PWR?" H 7250 6600 50  0001 C CNN
+F 1 "VCC" V 7265 6878 50  0000 L CNN
+F 2 "" H 7250 6750 50  0001 C CNN
+F 3 "" H 7250 6750 50  0001 C CNN
+	1    7250 6750
+	0    1    1    0
+$EndComp
+$Comp
+L power:Earth #PWR?
+U 1 1 61AD80DC
+P 7250 6850
+F 0 "#PWR?" H 7250 6600 50  0001 C CNN
+F 1 "Earth" H 7250 6700 50  0001 C CNN
+F 2 "" H 7250 6850 50  0001 C CNN
+F 3 "~" H 7250 6850 50  0001 C CNN
+	1    7250 6850
+	0    -1   -1   0
+$EndComp
+Wire Wire Line
+	5800 5850 5550 5850
+Wire Wire Line
+	5550 5950 5800 5950
+Wire Wire Line
+	5550 6150 5800 6150
+Wire Wire Line
+	5800 6250 5550 6250
+Wire Wire Line
+	5550 6350 5800 6350
+Wire Wire Line
+	5800 6450 5550 6450
+Wire Wire Line
+	5550 6550 5800 6550
+Wire Wire Line
+	5800 6650 5550 6650
+Wire Wire Line
+	5550 6750 5800 6750
+Wire Wire Line
+	5800 6850 5550 6850
 Wire Bus Line
 	11400 7000 14100 7000
@@
 Wire Bus Line
 	3400 4100 3400 6400
+Text Notes 5600 5850 0    50   ~ 0
+CLK
+Text Label 5600 5950 0    50   ~ 0
+DIO
+Text Label 5600 6150 0    50   ~ 0
+K2
+Text Label 5600 6250 0    50   ~ 0
+K1
+Text Label 5600 6350 0    50   ~ 0
+GRID1
+Text Label 5600 6450 0    50   ~ 0
+GRID2
+Text Label 5600 6550 0    50   ~ 0
+GRID3
+Text Label 5600 6650 0    50   ~ 0
+GRID4
+Text Label 5600 6750 0    50   ~ 0
+GRID5
+Text Label 5600 6850 0    50   ~ 0
+GRID6
 $EndSCHEMATC
