File: prinsip/prinsip.sch (KiCad schematic (older format))
At the start: 0 parts

Commit message: ЗАМЕЧАНИЕ
Parts:
- added SW1, SW2, SW3, SW4, SW5: SW_MEC_5G, symbol Switch:SW_MEC_5G
- added U? (x2): ATmega8515L-8JU, Package_LCC:PLCC-44, symbol MCU_Microchip_ATmega:ATmega8515L-8JU
- added U?: MCP23S17_SO, Package_SO:SOIC-28W_7.5x17.9mm_P1.27mm, symbol Interface_Expansion:MCP23S17_SO
- added U?: MAX232, symbol Interface_UART:MAX232
- added U?: 6264, symbol custom:6264
- added U?: 74LS373, symbol 74xx:74LS373
- added U?: HDSP-7401, Display_7Segment:HDSP-7401, symbol Display_Character:HDSP-7401
Connections:
- net labels added: Earth, XRAM_ADDR
- wire segments 0 -> 63
Other:
- note added: "Источник"
- note added: "Пульт оператора"

Commit message: Added prinsip
Parts:
- removed U?: HDSP-7401, Display_7Segment:HDSP-7401, symbol Display_Character:HDSP-7401
- added U?: CA56-12CGKWA, Display_7Segment:CA56-12CGKWA, symbol Display_Character:CA56-12CGKWA
- added U?: TM1637, DIP778W43P254L2612H431Q20N, symbol TM1637:TM1637
- U?: symbol custom:6264 -> prinsip-rescue:6264-custom
Connections:
- net labels added: VCC
- net labels removed: XRAM_ADDR
- wire segments 63 -> 109

Commit message: Updated code and PRINSIP
Parts:
- added C? (x2): 1мкФ, symbol Device:C
- added C? (x2): C, symbol Device:C
- added SW?: SW_MEC_5G-Switch, symbol prinsip-rescue:SW_MEC_5G-Switch
- added ZQ1, ZQ2: Resonator_Small, symbol Device:Resonator_Small
- SW1, SW2, SW3, SW4, SW5: symbol Switch:SW_MEC_5G -> prinsip-rescue:SW_MEC_5G-Switch
- U1: renamed from U?; symbol MCU_Microchip_ATmega:ATmega8515L-8JU -> prinsip-rescue:ATmega8515L-8JU-MCU_Microchip_ATmega
- U?: symbol Interface_Expansion:MCP23S17_SO -> prinsip-rescue:MCP23S17_SO-Interface_Expansion
- U?: symbol Interface_UART:MAX232 -> prinsip-rescue:MAX232-Interface_UART
- U?: symbol MCU_Microchip_ATmega:ATmega8515L-8JU -> prinsip-rescue:ATmega8515L-8JU-MCU_Microchip_ATmega
- U?: symbol 74xx:74LS373 -> prinsip-rescue:74LS373-74xx
- U?: symbol Display_Character:CA56-12CGKWA -> prinsip-rescue:CA56-12CGKWA-Display_Character
- U?: symbol TM1637:TM1637 -> prinsip-rescue:TM1637-TM1637
Connections:
- net labels removed: VCC
- wire segments 109 -> 171
Other:
- note added: "8МГц"
- note added: "С1\n22нФ"
- note added: "С2\n22нФ"
- moved on the sheet: U?

Commit message: Trying prinsip
Parts:
- removed SW?: SW_MEC_5G-Switch, symbol prinsip-rescue:SW_MEC_5G-Switch
- added SW2: SW_DPDT_x2, symbol Switch:SW_DPDT_x2
- added U?: USBAsp, symbol prinsip-rescue:USBASP
- gave numbers to parts that had none: 7
Connections:
- new net: SW2.2 (B), U?.SCK
Other:
- note added: "#"
- note added: "1"
- note added: "2"
- note added: "A10"
- note added: "A11"
- note added: "A12"
- note added: "A13"
- note added: "A14"
- note added: "A15"
- note added: "A8"
- note added: "A9"
- note added: "BTN0"
- note added: "BTN1"
- note added: "BTN2"
- note added: "BTN3"
- note added: "BTN4"
- note added: "D0"
- note added: "D1"
- note added: "D1\n"
- note added: "D2"
- note added: "D3"
- note added: "D4"
- note added: "D5"
- note added: "D6"
- note added: "D7"
- note added: "DIO"
- note added: "G1"
- note added: "G2"
- note added: "G3"
- note added: "G4"
- note added: "GND"
- note added: "LE"
- note added: "MISO"
- note added: "MOSI"
- note added: "MOSI\n"
- note added: "PING"
- note added: "PONG"
- note added: "Q0/A8"
- note added: "Q1/A9"
- note added: "Q2/A10"
- note added: "Q3/A11"
- note added: "Q4/A12"
- note added: "Q5/A13"
- note added: "Q6/A14"
- note added: "Q7/A15"
- note added: "RCVD"
- note added: "RST"
- note added: "SCK_RC"
- note added: "SCK_TR"
- note added: "SS"
- note added: "THR1_0"
- note added: "THR1_1"
- note added: "THR1_2"
- note added: "THR1_3"
- note added: "THR1_4"
- note added: "THR1_5"
- note added: "THR1_6"
- note added: "THR1_7"
- note added: "THR2_0"
- note added: "THR2_1"
- note added: "THR2_2"
- note added: "THR2_3"
- note added: "THR2_4"
- note added: "THR2_5"
- note added: "THR2_6"
- note added: "THR2_7"
- note added: "TM_CLK"
- note added: "TXD"
- note added: "VCC"
- note added: "VCC / +5В"
- note added: "a"
- note added: "b"
- note added: "c"
- note added: "d"
- note added: "dp"
- note added: "e"
- note added: "f"
- note added: "g"
- note added: "~RD"
- note added: "~SS"
- note added: "~WR"
- note added: "К RXD ПЭВМ"
- note added: "Назначение"
- note added: "Получатель"

Commit message: update prinsip
Parts:
- SW1: value SW_MEC_5G -> Выбрать канал 1
- SW2: value SW_MEC_5G -> Выбрать канал 2
- SW3: value SW_MEC_5G -> Выбрать канал 3
- SW4: value SW_MEC_5G -> Выбрать канал 4
- SW5: value SW_MEC_5G -> Выбрать канал 5
Changed lines of the file:
@@
 P 7600 8950
 F 0 "SW1" H 7600 9235 50  0000 C CNN
-F 1 "SW_MEC_5G" H 7600 9144 50  0000 C CNN
+F 1 "Выбрать канал 1" H 7600 9144 50  0000 C CNN
 F 2 "" H 7600 9150 50  0001 C CNN
 F 3 "http://www.apem.com/int/index.php?controller=attachment&id_attachment=488" H 7600 9150 50  0001 C CNN
@@
 P 7600 9300
 F 0 "SW2" H 7600 9585 50  0000 C CNN
-F 1 "SW_MEC_5G" H 7600 9494 50  0000 C CNN
+F 1 "Выбрать канал 2" H 7600 9494 50  0000 C CNN
 F 2 "" H 7600 9500 50  0001 C CNN
 F 3 "http://www.apem.com/int/index.php?controller=attachment&id_attachment=488" H 7600 9500 50  0001 C CNN
@@
 P 7600 9650
 F 0 "SW3" H 7600 9935 50  0000 C CNN
-F 1 "SW_MEC_5G" H 7600 9844 50  0000 C CNN
+F 1 "Выбрать канал 3" H 7600 9844 50  0000 C CNN
 F 2 "" H 7600 9850 50  0001 C CNN
 F 3 "http://www.apem.com/int/index.php?controller=attachment&id_attachment=488" H 7600 9850 50  0001 C CNN
@@
 P 7600 10000
 F 0 "SW4" H 7600 10285 50  0000 C CNN
-F 1 "SW_MEC_5G" H 7600 10194 50  0000 C CNN
+F 1 "Выбрать канал 4" H 7600 10194 50  0000 C CNN
 F 2 "" H 7600 10200 50  0001 C CNN
 F 3 "http://www.apem.com/int/index.php?controller=attachment&id_attachment=488" H 7600 10200 50  0001 C CNN
@@
 P 7600 10350
 F 0 "SW5" H 7600 10635 50  0000 C CNN
-F 1 "SW_MEC_5G" H 7600 10544 50  0000 C CNN
+F 1 "Выбрать канал 5" H 7600 10544 50  0000 C CNN
 F 2 "" H 7600 10550 50  0001 C CNN
 F 3 "http://www.apem.com/int/index.php?controller=attachment&id_attachment=488" H 7600 10550 50  0001 C CNN
@@
 Text Notes 14450 3500 0    50   ~ 0
 GND
-Wire Bus Line
-	8900 7800 8900 8300
 $Comp
 L prinsip-rescue:USBASP U?
@@
 Wire Wire Line
 	14850 2450 14850 2600
-Wire Bus Line
-	9150 5350 9150 5650
-Wire Bus Line
-	6350 6750 10050 6750
-Wire Bus Line
-	12600 4450 14350 4450
-Wire Bus Line
-	15950 1800 15950 3000
-Wire Bus Line
-	6850 8550 6850 10800
-Wire Bus Line
-	2550 1800 2550 10850
-Wire Bus Line
-	8800 7400 8800 10800
-Wire Bus Line
-	12600 1600 12600 5950
-Wire Bus Line
-	4200 8550 4200 10850
-Wire Bus Line
-	14350 1800 14350 4450
-Wire Bus Line
-	6350 1800 6350 6750
-Wire Bus Line
-	10050 1600 10050 6750
 Text Notes 14450 2600 0    50   ~ 0
 RST
+Wire Bus Line
+	9150 5350 9150 5650
+Wire Bus Line
+	6350 6750 10050 6750
+Wire Bus Line
+	12600 4450 14350 4450
+Wire Bus Line
+	8900 7800 8900 8300
+Wire Bus Line
+	15950 1800 15950 3000
+Wire Bus Line
+	6850 8550 6850 10800
+Wire Bus Line
+	2550 1800 2550 10850
+Wire Bus Line
+	8800 7400 8800 10800
+Wire Bus Line
+	12600 1600 12600 5950
+Wire Bus Line
+	4200 8550 4200 10850
+Wire Bus Line
+	14350 1800 14350 4450
+Wire Bus Line
+	6350 1800 6350 6750
+Wire Bus Line
+	10050 1600 10050 6750
 $EndSCHEMATC
